File: PCB_CAD/PCB_Order2/PCB_Order2.kicad_pcb (KiCad board)
At the start: 4 copper layers, 105.5 x 59.5 mm, 48 parts

Commit message: pcb'd dix9211 and lss with power
Parts:
- LLS In1: moved to F.Cu
- SPDIFTX1: moved to F.Cu
- dixSupply_bulk1, dixSupply_noise1: moved to B.Cu
- moved dixSupply_bulk1 176.5 mm to (250.5, 143.3), turned to 90 degrees
- moved dixSupply_noise1 173.4 mm to (248.4, 143.5), turned to 90 degrees
- moved DigitalOut1 138.6 mm to (249.9, 161.8)
- moved SpdifOut_ImpedanceMatch1 131.1 mm to (255.8, 158.5)
- moved SpdifOut_AcCoupling1 128.7 mm to (254.4, 155.9), turned to 0 degrees
- moved llsOut_refLo_noise2 126.1 mm to (247.7, 154.9)
- moved LLS Out1 125.4 mm to (251.3, 153.7)
- moved R3 122.4 mm to (241.5, 163.1), turned to -90 degrees
- moved R2 121.8 mm to (241.5, 159.6), turned to -90 degrees
- moved llsOut_refHi_noise2 121.4 mm to (250.7, 150.0), turned to -90 degrees
- moved SPDIFTX1 109.9 mm to (250.2, 151.5)
- moved LLS In1 6.27 mm to (107.8, 138.6), turned to 0 degrees
- moved DAC1 0.08 mm to (177.3, 106.7)
Connections:
- uController1 pad 69: unconnected-(uController1-PB10-Pad69) -> /I2S2_CK
- uController1 pad 73: unconnected-(uController1-PB12-Pad73) -> /I2S2_WS
- uController1 pad 96: unconnected-(uController1-PC6-Pad96) -> /I2S2_MCK
Routing:
- net /I2S2_MCK: track 0.00 -> 125.9 mm, vias 0 -> 3
- net /I2S3_WS: track 0.00 -> 85.2 mm, vias 0 -> 5
- net /I2S2_WS: track 0.00 -> 85.0 mm, vias 0 -> 3
- net /I2S3_SDO: track 0.00 -> 73.5 mm, vias 0 -> 3
- net /I2S2_CK: track 0.00 -> 70.4 mm, vias 0 -> 3
- net /I2S2_SDO: track 0.00 -> 67.9 mm, vias 0 -> 3
- net /I2S3_MCK: track 0.00 -> 36.6 mm, vias 0 -> 1
- net /I2C1_SDA: track 0.00 -> 33.6 mm, vias 0 -> 1
- net /I2C1_SCL: track 0.00 -> 32.7 mm, vias 0 -> 1
- net /I2S3_CK: track 0.00 -> 31.8 mm, vias 0 -> 3
- net GNDD: track 0.00 -> 20.1 mm, vias 3 -> 8
- net VDD_DIV: track 4.59 -> 15.8 mm, vias 0 -> 1
- net VDD: track 4.67 -> 14.9 mm, vias 1 -> 4
- net Net-(DigitalOut1-Pad2): track 0.00 -> 7.59 mm
- net /SPDIFTX_OUT: track 0.00 -> 5.28 mm, vias 0 -> 1
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Other:
- board text added: "note: we know better than TI here"

Commit message: dac power and digital out done
Parts:
- removed DacMute_CurrentLimit1: 10k, Resistor_SMD:R_0603_1608Metric_Pad0.98x0.95mm_HandSolder
- Dac_ChargePump_cap1, ImpMatching_LLSin1, dacVref_bypass1: moved to B.Cu
- LLS In1: moved to B.Cu
- moved llsOut_refHi_noise1 157.3 mm to (226.6, 153.3)
- moved DigitalIn1 131.7 mm to (227.6, 158.3)
- moved llsOut_refLo_noise1 129.5 mm to (235.3, 152.0), turned to 90 degrees
- moved LLS In1 124.4 mm to (231.4, 152.4)
- moved LLSin_ACcouple1 118.4 mm to (228.2, 156.4)
- moved ImpMatching_LLSin1 108.1 mm to (225.3, 156.1), turned to 180 degrees
- moved DacAnalogSupply_bulk1 104.4 mm to (180.9, 102.9)
- moved DacAnalogSupply_noise1 104.1 mm to (180.9, 104.9), turned to 180 degrees
- moved DacOut_L_res1 93.4 mm to (166.0, 130.1)
- moved DacOut_L_decouple1 93.4 mm to (166.3, 115.8)
- moved DacOut_R_res1 93.4 mm to (166.0, 132.6)
- moved DacOut_R_decouple1 93.4 mm to (166.3, 118.8)
- moved Dac_ChargePump_Decouple1 87.9 mm to (166.9, 104.2), turned to 180 degrees
- moved Dac_ChargePump_cap1 87.7 mm to (167.7, 102.8), turned to 90 degrees
- moved Dac_DigitalSup_bulk2 84.4 mm to (165.7, 99.3), turned to 90 degrees
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Connections:
- DAC1 pad 4: Net-(DAC1-MUTEB) -> VDD
- uController1 pad 1: unconnected-(uController1-PE2-Pad1) -> /KP_Col5
- uController1 pad 123: unconnected-(uController1-PD7-Pad123) -> /SPDIFRX_IN0
- uController1 pad 2: unconnected-(uController1-PE3-Pad2) -> /KP_Col4
- uController1 pad 3: unconnected-(uController1-PE4-Pad3) -> /KP_Row1
- uController1 pad 4: unconnected-(uController1-PE5-Pad4) -> /KP_Col3
- uController1 pad 5: unconnected-(uController1-PE6-Pad5) -> /KP_Row2
- uController1 pad 7: unconnected-(uController1-PC13-Pad7) -> /KP_Row3
- uController1 pad 8: unconnected-(uController1-PC14-Pad8) -> /KP_Col2
- uController1 pad 9: unconnected-(uController1-PC15-Pad9) -> /KP_Col1
Routing:
- net (no net): track 5644.8 -> 0.00 mm
- net GNDD: track 20.1 -> 82.4 mm, vias 8 -> 33
- net /SPDIFRX_IN0: track 0.00 -> 19.1 mm
- net Net-(DAC1-LINEVDD): track 0.00 -> 11.1 mm
- net VDD: track 14.9 -> 24.2 mm, vias 4 -> 7
- net Net-(DAC1-VDDA): track 0.00 -> 7.10 mm
- net VDD_DIV: track 15.8 -> 22.6 mm
- net Net-(LLS In1-B): track 0.00 -> 6.65 mm
- net /I2S2_MCK: track 125.9 -> 132.0 mm
- net Net-(DigitalIn1-Pad2): track 0.00 -> 5.37 mm
- net GNDA: track 0.00 -> 4.61 mm, vias 0 -> 3
- net /I2S2_WS: track 85.0 -> 81.3 mm
- net Net-(DAC1-VREF): track 0.00 -> 3.37 mm, vias 0 -> 1
- net /I2S2_CK: track 70.4 -> 73.7 mm
- net /I2S2_SDO: track 67.9 -> 64.6 mm
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