File: PCB_CAD/PCB_Order2/PCB_Order2.kicad_pcb (KiCad board)
At the start: 4 copper layers, 105.5 x 59.5 mm, 47 parts

Commit message: updating things
Parts:
- DacOut_L_decouple1, DacOut_L_res1, DacOut_R_decouple1, DacOut_R_res1: moved to B.Cu
- moved C2 96.5 mm to (161.2, 93.7)
- moved C3 96.2 mm to (161.2, 95.7)
- moved AnalogOut1 75.3 mm to (191.6, 154.5), turned to -90 degrees
- moved DacOut_L_decouple1 55.1 mm to (212.8, 145.3)
- moved DacOut_R_decouple1 41.5 mm to (198.0, 145.5)
- moved AnalogIn1 33.6 mm to (161.8, 154.4), turned to -90 degrees
- moved DacOut_R_res1 25.6 mm to (172.1, 107.7), turned to -90 degrees
- moved DacOut_L_res1 22.0 mm to (170.5, 108.6), turned to -90 degrees
Routing:
- net Net-(AnalogOut1-Pad3): track 0.00 -> 86.7 mm, vias 0 -> 2
- net Net-(AnalogOut1-Pad2): track 0.00 -> 70.9 mm, vias 0 -> 2
- net Net-(AnalogIn1-Pad3): track 0.00 -> 67.4 mm, vias 0 -> 1
- net Net-(AnalogIn1-Pad2): track 0.00 -> 67.0 mm, vias 0 -> 1
- net Net-(ADC1-RIN): track 0.00 -> 8.79 mm
- net Net-(ADC1-LIN): track 0.00 -> 8.55 mm
- net Net-(DAC1-RLINEOUT): track 0.00 -> 3.50 mm, vias 0 -> 1
- net Net-(DAC1-LLINEOU): track 0.00 -> 2.27 mm, vias 0 -> 1
- net GNDD: track 82.4 -> 84.0 mm, vias 33 -> 34
