File: PCB_CAD/PCB_Order2/PCB_Order2.kicad_pcb (KiCad board)
At the start: 4 copper layers, 105.5 x 59.5 mm, 58 parts

Commit message: pinned out adc power filtering and header for the keypad
Parts:
- removed C2, C3: 10uF, Capacitor_SMD:C_0805_2012Metric_Pad1.18x1.45mm_HandSolder
- moved K1 174.5 mm to (175.0, 135.8), turned to 180 degrees
- moved adc_L_acCouple1 34.4 mm to (161.2, 95.6)
- moved adc_R_acCouple1 33.1 mm to (161.2, 93.6)
- moved DigitalOut1 18.1 mm to (241.9, 175.9)
- moved DigitalIn1 17.6 mm to (226.8, 175.9)
- moved DacOut_L_decouple1 15.4 mm to (212.7, 160.7)
- moved AnalogIn1 15.2 mm to (161.7, 169.6)
- moved AnalogOut1 15.1 mm to (191.5, 169.6)
- moved DacOut_R_decouple1 15.1 mm to (198.0, 160.6)
Routing:
- net /KP_Col1: track 0.00 -> 70.8 mm, vias 0 -> 2
- net /KP_Col2: track 0.00 -> 70.1 mm, vias 0 -> 2
- net /KP_Row2: track 0.00 -> 69.4 mm, vias 0 -> 2
- net /KP_Row3: track 0.00 -> 69.3 mm, vias 0 -> 2
- net /KP_Col3: track 0.00 -> 68.6 mm, vias 0 -> 2
- net /KP_Row1: track 0.00 -> 67.8 mm, vias 0 -> 2
- net /KP_Row4: track 0.00 -> 66.4 mm, vias 0 -> 5
- net /KP_Col4: track 0.00 -> 63.8 mm, vias 0 -> 2
- net /KP_Col5: track 0.00 -> 63.3 mm, vias 0 -> 2
- net Net-(DigitalOut1-Pad2): track 7.59 -> 26.9 mm
- net Net-(DigitalIn1-Pad2): track 5.37 -> 23.3 mm
- net Net-(AnalogIn1-Pad2): track 67.0 -> 82.2 mm
- net Net-(AnalogIn1-Pad3): track 67.4 -> 82.5 mm
- net /I2S3_WS: track 85.2 -> 99.1 mm
- net /I2S1_WS: track 112.8 -> 124.0 mm
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
Commit message: added footprints to schematic
Parts:
- added DbC1: 15u, Capacitor_SMD:C_0805_2012Metric_Pad1.18x1.45mm_HandSolder, F.Cu at (80.7, 91.9)
- added DnC1: 0.15u, Capacitor_SMD:C_0805_2012Metric_Pad1.18x1.45mm_HandSolder, F.Cu at (80.7, 94.9)
- added FbC1: 15u, Capacitor_SMD:C_0805_2012Metric_Pad1.18x1.45mm_HandSolder, F.Cu at (80.7, 97.9)
- added FbC2: 15u, Capacitor_SMD:C_0805_2012Metric_Pad1.18x1.45mm_HandSolder, F.Cu at (80.7, 100.9)
- added FnC1: 0.15u, Capacitor_SMD:C_0805_2012Metric_Pad1.18x1.45mm_HandSolder, F.Cu at (80.7, 103.9)
- added FnC2: 0.15u, Capacitor_SMD:C_0805_2012Metric_Pad1.18x1.45mm_HandSolder, F.Cu at (80.7, 106.9)
- added LC1: ~, Connector_PinSocket_2.54mm:PinSocket_1x04_P2.54mm_Vertical, F.Cu at (104.6, 92.7)
- added MbC1: 15u, Capacitor_SMD:C_0805_2012Metric_Pad1.18x1.45mm_HandSolder, F.Cu at (80.7, 109.9)
- added MbC2: 15u, Capacitor_SMD:C_0805_2012Metric_Pad1.18x1.45mm_HandSolder, F.Cu at (80.7, 112.9)
- added MbC3: 15u, Capacitor_SMD:C_0805_2012Metric_Pad1.18x1.45mm_HandSolder, F.Cu at (85.5, 91.9)
- added MbC4: 15u, Capacitor_SMD:C_0805_2012Metric_Pad1.18x1.45mm_HandSolder, F.Cu at (85.5, 94.9)
- added MbC5: 15u, Capacitor_SMD:C_0805_2012Metric_Pad1.18x1.45mm_HandSolder, F.Cu at (85.5, 97.9)
- added MbC6: 15u, Capacitor_SMD:C_0805_2012Metric_Pad1.18x1.45mm_HandSolder, F.Cu at (85.5, 100.9)
- added MbC7: 15u, Capacitor_SMD:C_0805_2012Metric_Pad1.18x1.45mm_HandSolder, F.Cu at (85.5, 103.9)
- added MbC8: 15u, Capacitor_SMD:C_0805_2012Metric_Pad1.18x1.45mm_HandSolder, F.Cu at (85.5, 106.9)
- added MbC9: 15u, Capacitor_SMD:C_0805_2012Metric_Pad1.18x1.45mm_HandSolder, F.Cu at (85.5, 109.9)
- added MnC1: 0.15u, Capacitor_SMD:C_0805_2012Metric_Pad1.18x1.45mm_HandSolder, F.Cu at (85.5, 112.9)
- added MnC2: 0.15u, Capacitor_SMD:C_0805_2012Metric_Pad1.18x1.45mm_HandSolder, F.Cu at (90.3, 91.9)
- added MnC3: 0.15u, Capacitor_SMD:C_0805_2012Metric_Pad1.18x1.45mm_HandSolder, F.Cu at (90.3, 94.9)
- added MnC4: 0.15u, Capacitor_SMD:C_0805_2012Metric_Pad1.18x1.45mm_HandSolder, F.Cu at (90.3, 97.9)
- added MnC5: 0.15u, Capacitor_SMD:C_0805_2012Metric_Pad1.18x1.45mm_HandSolder, F.Cu at (90.3, 100.9)
- added MnC6: 0.15u, Capacitor_SMD:C_0805_2012Metric_Pad1.18x1.45mm_HandSolder, F.Cu at (90.3, 103.9)
- added MnC7: 0.15u, Capacitor_SMD:C_0805_2012Metric_Pad1.18x1.45mm_HandSolder, F.Cu at (90.3, 106.9)
- added MnC8: 0.15u, Capacitor_SMD:C_0805_2012Metric_Pad1.18x1.45mm_HandSolder, F.Cu at (90.3, 109.9)
- added MnC9: 0.15u, Capacitor_SMD:C_0805_2012Metric_Pad1.18x1.45mm_HandSolder, F.Cu at (90.3, 112.9)
- added RB1: 600, Resistor_SMD:R_0603_1608Metric_Pad0.98x0.95mm_HandSolder, F.Cu at (104.5, 103.9)
- added RB2: 600, Resistor_SMD:R_0603_1608Metric_Pad0.98x0.95mm_HandSolder, F.Cu at (104.5, 106.4)
- added RB3: 600, Resistor_SMD:R_0603_1608Metric_Pad0.98x0.95mm_HandSolder, F.Cu at (104.5, 108.9)
- added RB4: 600, Resistor_SMD:R_0603_1608Metric_Pad0.98x0.95mm_HandSolder, F.Cu at (104.5, 111.4)
- added RbC1: 15u, Capacitor_SMD:C_0805_2012Metric_Pad1.18x1.45mm_HandSolder, F.Cu at (95.1, 91.9)
- added RbC2: 15u, Capacitor_SMD:C_0805_2012Metric_Pad1.18x1.45mm_HandSolder, F.Cu at (95.1, 94.9)
- added RbC3: 15u, Capacitor_SMD:C_0805_2012Metric_Pad1.18x1.45mm_HandSolder, F.Cu at (95.1, 97.9)
- added RbC4: 15u, Capacitor_SMD:C_0805_2012Metric_Pad1.18x1.45mm_HandSolder, F.Cu at (95.1, 100.9)
- added RbC5: 15u, Capacitor_SMD:C_0805_2012Metric_Pad1.18x1.45mm_HandSolder, F.Cu at (95.1, 103.9)
- added RbC6: 15u, Capacitor_SMD:C_0805_2012Metric_Pad1.18x1.45mm_HandSolder, F.Cu at (95.1, 106.9)
- added RbC7: 15u, Capacitor_SMD:C_0805_2012Metric_Pad1.18x1.45mm_HandSolder, F.Cu at (95.1, 109.9)
- added RnC1: 0.15u, Capacitor_SMD:C_0805_2012Metric_Pad1.18x1.45mm_HandSolder, F.Cu at (95.1, 112.9)
- added RnC2: 0.15u, Capacitor_SMD:C_0805_2012Metric_Pad1.18x1.45mm_HandSolder, F.Cu at (99.9, 91.9)
- added RnC3: 0.15u, Capacitor_SMD:C_0805_2012Metric_Pad1.18x1.45mm_HandSolder, F.Cu at (99.9, 94.9)
- added RnC4: 0.15u, Capacitor_SMD:C_0805_2012Metric_Pad1.18x1.45mm_HandSolder, F.Cu at (99.9, 97.9)
- added RnC5: 0.15u, Capacitor_SMD:C_0805_2012Metric_Pad1.18x1.45mm_HandSolder, F.Cu at (99.9, 100.9)
- added RnC6: 0.15u, Capacitor_SMD:C_0805_2012Metric_Pad1.18x1.45mm_HandSolder, F.Cu at (99.9, 103.9)
- added RnC7: 0.15u, Capacitor_SMD:C_0805_2012Metric_Pad1.18x1.45mm_HandSolder, F.Cu at (99.9, 106.9)
Connections:
- RAM1 pad 3: VCCQ -> Net-(RAM1-VDDQ_1)
- RAM1 pad 43: VCCQ -> Net-(RAM1-VDDQ_3)
- RAM1 pad 49: VCCQ -> Net-(RAM1-VDDQ_4)
- RAM1 pad 9: VCCQ -> Net-(RAM1-VDDQ_2)
- uController1 pad 108: unconnected-(uController1-VDD-Pad108) -> VDD
- uController1 pad 121: unconnected-(uController1-VDDMMC-Pad121) -> VDD
- uController1 pad 131: unconnected-(uController1-VDD-Pad131) -> VDD
- uController1 pad 17: unconnected-(uController1-VDD-Pad17) -> VDD
- uController1 pad 30: unconnected-(uController1-VDD-Pad30) -> VDD
- uController1 pad 39: unconnected-(uController1-VDD-Pad39) -> VDD
- uController1 pad 52: unconnected-(uController1-VDD-Pad52) -> VDD
- uController1 pad 62: unconnected-(uController1-VDD-Pad62) -> VDD
- uController1 pad 69: /I2S2_CK -> /I2C2_SCL
- uController1 pad 70: unconnected-(uController1-PB11-Pad70) -> /I2C2_SDA
- uController1 pad 72: unconnected-(uController1-VDD-Pad72) -> VDD
- uController1 pad 74: unconnected-(uController1-PB13-Pad74) -> /I2S2_CK
- uController1 pad 84: unconnected-(uController1-VDD-Pad84) -> VDD
