File: PCB_CAD/PCB_Order2/PCB_Order2.kicad_sch (KiCad schematic)
At the start: 51 parts

Commit message: added footprints
Parts:
- adcBead1: renamed from adcBead; footprint (none) -> Resistor_SMD:R_0603_1608Metric
- adcReset_rc_cap1: renamed from adcReset_rc_cap; footprint (none) -> Capacitor_SMD:C_0805_2012Metric_Pad1.18x1.45mm_HandSolder
- adcReset_rc_res1: renamed from adcReset_rc_res; footprint (none) -> Resistor_SMD:R_0603_1608Metric_Pad0.98x0.95mm_HandSolder
- adc_L_acCouple1: renamed from adc_L_acCouple; footprint (none) -> Capacitor_SMD:C_0805_2012Metric_Pad1.18x1.45mm_HandSolder
- adc_R_acCouple1: renamed from adc_R_acCouple; footprint (none) -> Capacitor_SMD:C_0805_2012Metric_Pad1.18x1.45mm_HandSolder
- adc_aSupply_bulk1: renamed from adc_aSupply_bulk; footprint (none) -> Capacitor_SMD:C_0805_2012Metric_Pad1.18x1.45mm_HandSolder
- adc_aSupply_noise1: renamed from adc_aSupply_noise; footprint (none) -> Capacitor_SMD:C_0805_2012Metric_Pad1.18x1.45mm_HandSolder
- adc_dSupply_bulk1, adc_dSupply_noise1: footprint (none) -> Capacitor_SMD:C_0805_2012Metric_Pad1.18x1.45mm_HandSolder
- adc_rego1: renamed from adc_rego; footprint (none) -> Capacitor_SMD:C_0805_2012Metric_Pad1.18x1.45mm_HandSolder
- renumbered VdivHigh to VdivHigh1, VdivLow to VdivLow1, adc_vcom to adc_vcom1
Changed lines of the file:
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@@
 		(on_board yes)
 		(dnp no)
-		(property "Reference" "adcReset_rc_res"
+		(property "Reference" "adcReset_rc_res1"
 			(at 318.77 196.85 90)
 			(effects
@@
 			)
 		)
-		(property "Footprint" ""
+		(property "Footprint" "Resistor_SMD:R_0603_1608Metric_Pad0.98x0.95mm_HandSolder"
 			(at 318.77 203.2 0)
 			(effects
@@
 			(project ""
 				(path "/85a2a93a-53e0-46c8-b7f5-ee661b6f3053"
-					(reference "adcReset_rc_res")
+					(reference "adcReset_rc_res1")
 					(unit 1)
 				)
@@
 		(on_board yes)
 		(dnp no)
-		(property "Reference" "adcBead"
+		(property "Reference" "adcBead1"
 			(at 292.1 167.6018 0)
 			(effects
@@
 			)
 		)
-		(property "Footprint" ""
+		(property "Footprint" "Resistor_SMD:R_0603_1608Metric"
 			(at 287.782 168.91 90)
 			(effects
@@
 			(project ""
 				(path "/85a2a93a-53e0-46c8-b7f5-ee661b6f3053"
-					(reference "adcBead")
+					(reference "adcBead1")
 					(unit 1)
 				)
@@
 			)
 		)
-		(property "Footprint" ""
+		(property "Footprint" "Capacitor_SMD:C_0805_2012Metric_Pad1.18x1.45mm_HandSolder"
 			(at 304.8 177.8 0)
 			(effects
@@
 		(on_board yes)
 		(dnp no)
-		(property "Reference" "VdivLow"
+		(property "Reference" "VdivLow1"
 			(at 459.74 132.08 90)
 			(effects
@@
 			(project "PCB_Order2"
 				(path "/85a2a93a-53e0-46c8-b7f5-ee661b6f3053"
-					(reference "VdivLow")
+					(reference "VdivLow1")
 					(unit 1)
 				)
@@
 		(on_board yes)
 		(dnp no)
-		(property "Reference" "adc_aSupply_bulk"
+		(property "Reference" "adc_aSupply_bulk1"
 			(at 294.64 172.2881 0)
 			(effects
@@
 			)
 		)
-		(property "Footprint" ""
+		(property "Footprint" "Capacitor_SMD:C_0805_2012Metric_Pad1.18x1.45mm_HandSolder"
 			(at 292.1 173.99 0)
 			(effects
@@
 			(project ""
 				(path "/85a2a93a-53e0-46c8-b7f5-ee661b6f3053"
-					(reference "adc_aSupply_bulk")
+					(reference "adc_aSupply_bulk1")
 					(unit 1)
 				)
@@
 		(on_board yes)
 		(dnp no)
-		(property "Reference" "adc_aSupply_noise"
+		(property "Reference" "adc_aSupply_noise1"
 			(at 294.6463 173.99 90)
 			(effects
@@
 			)
 		)
-		(property "Footprint" ""
+		(property "Footprint" "Capacitor_SMD:C_0805_2012Metric_Pad1.18x1.45mm_HandSolder"
 			(at 294.64 180.34 0)
 			(effects
@@
 			(project ""
 				(path "/85a2a93a-53e0-46c8-b7f5-ee661b6f3053"
-					(reference "adc_aSupply_noise")
+					(reference "adc_aSupply_noise1")
 					(unit 1)
 				)
@@
 		(dnp no)
 		(fields_autoplaced yes)
-		(property "Reference" "adc_rego"
+		(property "Reference" "adc_rego1"
 			(at 284.48 215.4681 0)
 			(effects
@@
 			)
 		)
-		(property "Footprint" ""
+		(property "Footprint" "Capacitor_SMD:C_0805_2012Metric_Pad1.18x1.45mm_HandSolder"
 			(at 281.94 217.17 0)
 			(effects
@@
 			(project ""
 				(path "/85a2a93a-53e0-46c8-b7f5-ee661b6f3053"
-					(reference "adc_rego")
+					(reference "adc_rego1")
 					(unit 1)
 				)
@@
 		(on_board yes)
 		(dnp no)
-		(property "Reference" "VdivHigh"
+		(property "Reference" "VdivHigh1"
 			(at 444.5 132.08 90)
 			(effects
@@
 			(project ""
 				(path "/85a2a93a-53e0-46c8-b7f5-ee661b6f3053"
-					(reference "VdivHigh")
+					(reference "VdivHigh1")
 					(unit 1)
 				)
@@
 			)
 		)
-		(property "Footprint" ""
+		(property "Footprint" "Capacitor_SMD:C_0805_2012Metric_Pad1.18x1.45mm_HandSolder"
 			(at 307.34 171.45 0)
 			(effects
@@
 		(dnp no)
 		(fields_autoplaced yes)
-		(property "Reference" "adc_vcom"
+		(property "Reference" "adc_vcom1"
 			(at 281.9463 201.93 90)
 			(effects
@@
 			(project ""
 				(path "/85a2a93a-53e0-46c8-b7f5-ee661b6f3053"
-					(reference "adc_vcom")
+					(reference "adc_vcom1")
 					(unit 1)
 				)
@@
 		(on_board yes)
 		(dnp no)
-		(property "Reference" "adc_L_acCouple"
+		(property "Reference" "adc_L_acCouple1"
 			(at 277.6982 191.77 90)
 			(effects
@@
 			)
 		)
-		(property "Footprint" ""
+		(property "Footprint" "Capacitor_SMD:C_0805_2012Metric_Pad1.18x1.45mm_HandSolder"
 			(at 278.13 198.12 0)
 			(effects
@@
 			(project ""
 				(path "/85a2a93a-53e0-46c8-b7f5-ee661b6f3053"
-					(reference "adc_L_acCouple")
+					(reference "adc_L_acCouple1")
 					(unit 1)
 				)
@@
 		(dnp no)
 		(fields_autoplaced yes)
-		(property "Reference" "adcReset_rc_cap"
+		(property "Reference" "adcReset_rc_cap1"
 			(at 340.36 204.0381 0)
 			(effects
@@
 			)
 		)
-		(property "Footprint" ""
+		(property "Footprint" "Capacitor_SMD:C_0805_2012Metric_Pad1.18x1.45mm_HandSolder"
 			(at 337.82 205.74 0)
 			(effects
@@
 			(project ""
 				(path "/85a2a93a-53e0-46c8-b7f5-ee661b6f3053"
-					(reference "adcReset_rc_cap")
+					(reference "adcReset_rc_cap1")
 					(unit 1)
 				)
@@
 		(on_board yes)
 		(dnp no)
-		(property "Reference" "adc_R_acCouple"
+		(property "Reference" "adc_R_acCouple1"
 			(at 277.6982 186.69 90)
 			(effects
@@
 			)
 		)
-		(property "Footprint" ""
+		(property "Footprint" "Capacitor_SMD:C_0805_2012Metric_Pad1.18x1.45mm_HandSolder"
 			(at 278.13 193.04 0)
 			(effects
@@
 			(project ""
 				(path "/85a2a93a-53e0-46c8-b7f5-ee661b6f3053"
-					(reference "adc_R_acCouple")
+					(reference "adc_R_acCouple1")
 					(unit 1)
 				)

Commit message: cubeMX and schematic add LCD, some work on RAM and ucontroller power
Parts:
- added DbC, FbC1, FbC2, RbC1, RbC2, RbC3, RbC4, RbC5, RbC6 (x2): 15u, symbol Device:C_Polarized_Small_US
- added DnC, FnC1, FnC2, RnC1, RnC2, RnC3, RnC4, RnC5, RnC6 (x2): 0.15u, symbol Device:C_Small
- added LC1: ~, Connector_PinSocket_2.54mm:PinSocket_1x04_P2.54mm_Vertical, symbol custom:GME12864
- added MbC1, MbC2, MbC3, MbC4, MbC5, MbC6, MbC7, MbC8, MbC9: 15u, Capacitor_SMD:C_0805_2012Metric_Pad1.18x1.45mm_HandSolder, symbol Device:C_Polarized_Small_US
- added MnC1, MnC2, MnC3, MnC4, MnC5, MnC6, MnC7, MnC8, MnC9: 0.15u, Capacitor_SMD:C_0805_2012Metric_Pad1.18x1.45mm_HandSolder, symbol Device:C_Small
- added RB1, RB2, RB3, RB4: 600, symbol Device:FerriteBead_Small
Connections:
- net GNDD: now also DbC.2, DnC.1, FbC1.2, FbC2.2, FnC1.1, FnC2.1, LC1.2 (GND), MbC1.2, MbC2.2, MbC3.2, MbC4.2, MbC5.2, MbC6.2, MbC7.2, MbC8.2, MbC9.2, MnC1.1, MnC2.2, MnC3.1, MnC4.1, MnC5.1, MnC6.1, MnC7.1, MnC8.1, MnC9.1, RbC1.2, RbC2.2, RbC3.2, RbC4.2, RbC5.2, RbC6.2, RbC6.2, RnC1.2, RnC2.1, RnC3.1, RnC4.1, RnC5.2, RnC6.1, RnC6.1
- net I2S2_CK: now also uController1.74 (PB13); no longer uController1.69 (PB10)
- net VDD: now also uController1.108 (VDD), uController1.121 (VDDMMC), uController1.131 (VDD), uController1.17 (VDD), uController1.30 (VDD), uController1.39 (VDD), uController1.52 (VDD), uController1.62 (VDD), uController1.72 (VDD), uController1.84 (VDD), DbC.1, DnC.2, FbC1.1, FbC2.1, FnC1.2, FnC2.2, LC1.1 (VCC), MbC1.1, MbC2.1, MbC3.1, MbC4.1, MbC5.1, MbC6.1, MbC7.1, MbC8.1, MbC9.1, MnC1.2, MnC2.1, MnC3.2, MnC4.2, MnC5.2, MnC6.2, MnC7.2, MnC8.2, MnC9.2, RB1.1, RB2.1, RB3.1, RB4.1, RbC1.1, RbC4.1, RbC5.1, RnC1.1, RnC4.2, RnC5.1
- net I2C2_SDA: now reaches uController1.70 (PB11)
- net I2C2_SDA: now also LC1.4 (SDA)
- removed net VCCQ: RAM1.3 (VDDQ_1), RAM1.43 (VDDQ_3), RAM1.49 (VDDQ_4), RAM1.9 (VDDQ_2)
- new net: RAM1.49 (VDDQ_4), RB4.2, RbC6.1, RnC6.2
- new net: RAM1.9 (VDDQ_2), RB2.2, RbC3.1, RnC3.2
- new net: RAM1.43 (VDDQ_3), RB3.2, RbC6.1, RnC6.2
- new net: RAM1.3 (VDDQ_1), RB1.2, RbC2.1, RnC2.2
- new net I2C2_SCL: LC1.3 (SCL), uController1.69 (PB10)
- no-connect marks 0 -> 30
Other:
- note added: "User IO"
- moved on the sheet: K1

Commit message: added footprints to schematic
Parts:
- DbC1: renamed from DbC; footprint (none) -> Capacitor_SMD:C_0805_2012Metric_Pad1.18x1.45mm_HandSolder
- DnC1: renamed from DnC; footprint (none) -> Capacitor_SMD:C_0805_2012Metric_Pad1.18x1.45mm_HandSolder
- FbC1, FbC2, FnC1, FnC2, RbC1, RbC2, RbC3, RbC4, RbC5, RbC6, RnC1, RnC2, RnC3, RnC4, RnC5, RnC6: footprint (none) -> Capacitor_SMD:C_0805_2012Metric_Pad1.18x1.45mm_HandSolder
- RB1, RB2, RB3, RB4: footprint (none) -> Resistor_SMD:R_0603_1608Metric_Pad0.98x0.95mm_HandSolder
- RbC7: renamed from RbC6; footprint (none) -> Capacitor_SMD:C_0805_2012Metric_Pad1.18x1.45mm_HandSolder
- RnC7: renamed from RnC6; footprint (none) -> Capacitor_SMD:C_0805_2012Metric_Pad1.18x1.45mm_HandSolder
Changed lines of the file:
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@@
 			)
 		)
-		(property "Footprint" ""
+		(property "Footprint" "Resistor_SMD:R_0603_1608Metric_Pad0.98x0.95mm_HandSolder"
 			(at 582.422 302.26 90)
 			(effects
@@
 			)
 		)
-		(property "Footprint" ""
+		(property "Footprint" "Capacitor_SMD:C_0805_2012Metric_Pad1.18x1.45mm_HandSolder"
 			(at 505.46 292.1 0)
 			(effects
@@
 			)
 		)
-		(property "Footprint" ""
+		(property "Footprint" "Resistor_SMD:R_0603_1608Metric_Pad0.98x0.95mm_HandSolder"
 			(at 488.442 311.15 90)
 			(effects
@@
 			)
 		)
-		(property "Footprint" ""
+		(property "Footprint" "Capacitor_SMD:C_0805_2012Metric_Pad1.18x1.45mm_HandSolder"
 			(at 664.21 325.12 0)
 			(effects
@@
 			)
 		)
-		(property "Footprint" ""
+		(property "Footprint" "Capacitor_SMD:C_0805_2012Metric_Pad1.18x1.45mm_HandSolder"
 			(at 598.17 330.2 0)
 			(effects
@@
 			)
 		)
-		(property "Footprint" ""
+		(property "Footprint" "Capacitor_SMD:C_0805_2012Metric_Pad1.18x1.45mm_HandSolder"
 			(at 497.84 358.14 0)
 			(effects
@@
 			)
 		)
-		(property "Footprint" ""
+		(property "Footprint" "Resistor_SMD:R_0603_1608Metric_Pad0.98x0.95mm_HandSolder"
 			(at 581.152 317.5 90)
 			(effects
@@
 			)
 		)
-		(property "Footprint" ""
+		(property "Footprint" "Capacitor_SMD:C_0805_2012Metric_Pad1.18x1.45mm_HandSolder"
 			(at 505.46 288.29 0)
 			(effects
@@
 			)
 		)
-		(property "Footprint" ""
+		(property "Footprint" "Resistor_SMD:R_0603_1608Metric_Pad0.98x0.95mm_HandSolder"
 			(at 489.712 294.64 90)
 			(effects
@@
 			)
 		)
-		(property "Footprint" ""
+		(property "Footprint" "Capacitor_SMD:C_0805_2012Metric_Pad1.18x1.45mm_HandSolder"
 			(at 594.36 330.2 0)
 			(effects
@@
 			)
 		)
-		(property "Footprint" ""
+		(property "Footprint" "Capacitor_SMD:C_0805_2012Metric_Pad1.18x1.45mm_HandSolder"
 			(at 497.84 353.06 0)
 			(effects
@@
 			)
 		)
-		(property "Footprint" ""
+		(property "Footprint" "Capacitor_SMD:C_0805_2012Metric_Pad1.18x1.45mm_HandSolder"
 			(at 491.49 326.39 0)
 			(effects
@@
 		(on_board yes)
 		(dnp no)
-		(property "Reference" "DbC"
+		(property "Reference" "DbC1"
 			(at 331.9018 289.56 90)
 			(effects
@@
 			)
 		)
-		(property "Footprint" ""
+		(property "Footprint" "Capacitor_SMD:C_0805_2012Metric_Pad1.18x1.45mm_HandSolder"
 			(at 331.47 295.91 0)
 			(effects
@@
 			(project ""
 				(path "/85a2a93a-53e0-46c8-b7f5-ee661b6f3053"
-					(reference "DbC")
+					(reference "DbC1")
 					(unit 1)
 				)
@@
 			)
 		)
-		(property "Footprint" ""
+		(property "Footprint" "Capacitor_SMD:C_0805_2012Metric_Pad1.18x1.45mm_HandSolder"
 			(at 664.21 328.93 0)
 			(effects
@@
 			)
 		)
-		(property "Footprint" ""
+		(property "Footprint" "Capacitor_SMD:C_0805_2012Metric_Pad1.18x1.45mm_HandSolder"
 			(at 496.57 326.39 0)
 			(effects
@@
 		(on_board yes)
 		(dnp no)
-		(property "Reference" "RnC6"
+		(property "Reference" "RnC7"
 			(at 576.58 320.0462 0)
 			(effects
@@
 			)
 		)
-		(property "Footprint" ""
+		(property "Footprint" "Capacitor_SMD:C_0805_2012Metric_Pad1.18x1.45mm_HandSolder"
 			(at 574.04 321.31 0)
 			(effects
@@
 			(project ""
 				(path "/85a2a93a-53e0-46c8-b7f5-ee661b6f3053"
-					(reference "RnC6")
+					(reference "RnC7")
 					(unit 1)
 				)
@@
 			)
 		)
-		(property "Footprint" ""
+		(property "Footprint" "Capacitor_SMD:C_0805_2012Metric_Pad1.18x1.45mm_HandSolder"
 			(at 499.11 313.69 0)
 			(effects
@@
 			)
 		)
-		(property "Footprint" ""
+		(property "Footprint" "Capacitor_SMD:C_0805_2012Metric_Pad1.18x1.45mm_HandSolder"
 			(at 575.31 306.07 0)
 			(effects
@@
 			)
 		)
-		(property "Footprint" ""
+		(property "Footprint" "Capacitor_SMD:C_0805_2012Metric_Pad1.18x1.45mm_HandSolder"
 			(at 495.3 313.69 0)
 			(effects
@@
 			)
 		)
-		(property "Footprint" ""
+		(property "Footprint" "Capacitor_SMD:C_0805_2012Metric_Pad1.18x1.45mm_HandSolder"
 			(at 495.3 298.45 0)
 			(effects
@@
 		(on_board yes)
 		(dnp no)
-		(property "Reference" "DnC"
+		(property "Reference" "DnC1"
 			(at 331.4763 293.37 90)
 			(effects
@@
 			)
 		)
-		(property "Footprint" ""
+		(property "Footprint" "Capacitor_SMD:C_0805_2012Metric_Pad1.18x1.45mm_HandSolder"
 			(at 331.47 299.72 0)
 			(effects
@@
 			(project ""
 				(path "/85a2a93a-53e0-46c8-b7f5-ee661b6f3053"
-					(reference "DnC")
+					(reference "DnC1")
 					(unit 1)
 				)
@@
 		(on_board yes)
 		(dnp no)
-		(property "Reference" "RbC6"
+		(property "Reference" "RbC7"
 			(at 580.39 320.4717 0)
 			(effects
@@
 			)
 		)
-		(property "Footprint" ""
+		(property "Footprint" "Capacitor_SMD:C_0805_2012Metric_Pad1.18x1.45mm_HandSolder"
 			(at 577.85 321.31 0)
 			(effects
@@
 			(project ""
 				(path "/85a2a93a-53e0-46c8-b7f5-ee661b6f3053"
-					(reference "RbC6")
+					(reference "RbC7")
 					(unit 1)
 				)
@@
 			)
 		)
-		(property "Footprint" ""
+		(property "Footprint" "Capacitor_SMD:C_0805_2012Metric_Pad1.18x1.45mm_HandSolder"
 			(at 499.11 298.45 0)
 			(effects
@@
 			)
 		)
-		(property "Footprint" ""
+		(property "Footprint" "Capacitor_SMD:C_0805_2012Metric_Pad1.18x1.45mm_HandSolder"
 			(at 579.12 306.07 0)
 			(effects

Commit message: schematic fixes and add USB, cubeMX update, add more useful documents
Parts:
- removed DacAnalogSupply_bead1: *TBD*, Resistor_SMD:R_0603_1608Metric, symbol Device:FerriteBead_Small
- removed DbC1, MbC1, MbC2, MbC3, MbC4, MbC5, MbC6, MbC7, MbC8, MbC9, dixSupply_bulk1: 15u, Capacitor_SMD:C_0805_2012Metric_Pad1.18x1.45mm_HandSolder, symbol Device:C_Polarized_Small_US
- removed adc_vcom1: 0.47u, Capacitor_SMD:C_0805_2012Metric_Pad1.18x1.45mm_HandSolder, symbol Device:C_Small
- added AcC1: 0.47u, symbol Device:C_Polarized_Small_US
- added DB1: 600, symbol Device:FerriteBead_Small
- added MnC10: 0.1u, Capacitor_SMD:C_0805_2012Metric_Pad1.18x1.45mm_HandSolder, symbol Device:C_Small
- added UR1: 33k, symbol Device:R_Small_US
- added UR2: 82k, symbol Device:R_Small_US
- added USB1: USB-M26FTU, CustomModels:USB-M26FTU, symbol USB-M26:USB-M26FTU
- AbC1: renamed from adc_aSupply_bulk1; value 15u -> 10u
- AbC2: renamed from adc_dSupply_bulk1; value 15u -> 10u
- AnC1: renamed from adc_aSupply_noise1; value 0.15u -> 0.1u
- AnC2: renamed from adc_dSupply_noise1; value 0.15u -> 0.1u
- ApC1: renamed from adcReset_rc_cap1; value 47u -> 4.7u
- LLS1: renamed from LLS In1
- LLS2: renamed from LLS Out1
- MnC1, MnC2, MnC3, MnC4, MnC5, MnC6, MnC7, MnC8, MnC9: value 0.15u -> 0.1u
- SPDIFR2: renamed from SpdifOut_ImpedanceMatch1; footprint Resistor_SMD:R_0603_1608Metric -> Resistor_SMD:R_0603_1608Metric_Pad0.98x0.95mm_HandSolder
- renumbered adcBead1 to AB1, adcReset_rc_res1 to AR1, adc_R_acCouple1 to AdbC1, adc_L_acCouple1 to AdbC2, adc_rego1 to ArC1, dixSupply_noise1 to DXnC1, K1 to KP1, llsOut_refHi_noise1 to LLSIC1, llsOut_refLo_noise1 to LLSIC2, llsOut_refHi_noise2 to LLSOC1, llsOut_refLo_noise2 to LLSOC2, DnC1 to LnC1, AnalogIn1 to RCAA1, AnalogOut1 to RCAA2, DigitalIn1 to RCAD1, DigitalOut1 to RCAD2, LLSin_ACcouple1 to SPDIFC1, SpdifOut_AcCoupling1 to SPDIFC2, ImpMatching_LLSin1 to SPDIFR1, VdivHigh1 to VDIVR1, VdivLow1 to VDIVR2
Connections:
- net GNDD: now also MnC1.2, MnC3.2, MnC4.2, MnC5.2, MnC6.2, MnC7.2, MnC8.2, MnC9.2, AcC1.2, MnC10.2, UR2.1; no longer MnC1.1, MnC3.1, MnC4.1, MnC5.1, MnC6.1, MnC7.1, MnC8.1, MnC9.1
- net VDD: now also AbC1.1, DacAnalogSupply_bulk1.1, MnC1.1, MnC3.1, MnC4.1, MnC5.1, MnC6.1, MnC7.1, MnC8.1, MnC9.1, uController1.144 (VDD), DB1.1, MnC10.1; no longer MnC1.2, MnC3.2, MnC4.2, MnC5.2, MnC6.2, MnC7.2, MnC8.2, MnC9.2, uController1.121 (VDDMMC)
- net at AB1.2, ADC1.5 (VA), AnC1.2: no longer AbC1.1
- net at DAC1.2 (VDDA), DacAnalogSupply_noise1.2: now also DB1.2; no longer DacAnalogSupply_bulk1.1
- net USB_OTG_HS_VBUS: now reaches uController1.101 (PA9)
- net USB_OTG_HS_VBUS: now also UR1.1, UR2.2
- net USB_OTG_HS_DM: now reaches uController1.103 (PA11)
- net USB_OTG_HS_DM: now also USB1.2
- net USB_OTG_HS_DP: now reaches uController1.104 (PA12)
- net USB_OTG_HS_DP: now also USB1.3
- net at ADC1.1 (VCOM): now also AcC1.1
- new net: UR1.2, USB1.1
- no-connect marks 30 -> 65

Commit message: schematic substantively complete (for real) (version 3.0) (final) (last)
Parts:
- removed Dac_ChargePump_bead1: 600, Resistor_SMD:R_0603_1608Metric, symbol Device:FerriteBead_Small
- removed Dac_DigitalSup_bulk1, Dac_DigitalSup_bulk2, FbC1, FbC2, RbC1, RbC2, RbC3, RbC4, RbC5, RbC6, RbC7: 15u, Capacitor_SMD:C_0805_2012Metric_Pad1.18x1.45mm_HandSolder, symbol Device:C_Polarized_Small_US
- removed RB1, RB2, RB3, RB4: 600, Resistor_SMD:R_0603_1608Metric_Pad0.98x0.95mm_HandSolder, symbol Device:FerriteBead_Small
- removed USB1: USB-M26FTU, CustomModels:USB-M26FTU, symbol USB-M26:USB-M26FTU
- added B1: PTS645SK43SMTR92LFS, CustomModels:SWITCH_45SK43SMTR92LFS, symbol red button:PTS645SK43SMTR92LFS
- added BC1, MunC1: 0.1u, symbol Device:C_Small
- added MR1: 100k, symbol Device:R_Small_US
- added MbC2: 1u, Capacitor_SMD:C_0805_2012Metric_Pad1.18x1.45mm_HandSolder, symbol Device:C_Small
- added MbC3, MbC4: 2.2u, Capacitor_SMD:C_0805_2012Metric_Pad1.18x1.45mm_HandSolder, symbol Device:C_Polarized_Small_US
- added MnC11, MnC12, MnC13: 0.1u, Capacitor_SMD:C_0805_2012Metric_Pad1.18x1.45mm_HandSolder, symbol Device:C_Small
- added MunC2: 1u, symbol Device:C_Small
- added SR1: 10k, symbol Device:R_Small_US
- added SW1: SLW-883935-2A-D, CustomModels:SLW-883935_CUD, symbol Same Sky slide switch:SLW-883935-2A-D
- added USB1: USB-M26FTR, CustomModels:USBM26FTR, symbol USB-M26FTR:USB-M26FTR
- AB1: footprint Resistor_SMD:R_0603_1608Metric -> Resistor_SMD:R_0603_1608Metric_Pad0.98x0.95mm_HandSolder
- AcC1: footprint (none) -> Capacitor_SMD:C_0805_2012Metric_Pad1.18x1.45mm_HandSolder
- AdbC1, AdbC2: symbol Device:C_Polarized_Small_US -> Device:C_Small
- renumbered ApC1 to AbC3, DacAnalogSupply_bulk1 to DbC1, Dac_ChargePump_cap1 to DcC1, Dac_ChargePump_Decouple1 to DcC2, DacAnalogSupply_noise1 to DnC1, dacVref_bypass1 to DrC1
Connections:
- net GNDD: now also B1.3, B1.4, BC1.2, MbC2.2, MbC3.2, MbC4.2, MnC11.1, MnC12.2, MnC13.2, MunC1.2, MunC2.2, SW1.3
- net USB_OTG_HS_DM: now also USB1.2
- net USB_OTG_HS_DP: now also USB1.3
- net VDD: now also DAC1.10 (LINEVDD), Dac_DigitalSup_noise1.1, RAM1.3 (VDDQ_1), RAM1.43 (VDDQ_3), RAM1.49 (VDDQ_4), RAM1.9 (VDDQ_2), RnC2.2, RnC3.2, RnC6.2, RnC7.2, uController1.121 (VDDMMC), uController1.143 (PDR_ON), uController1.33 (VDDA), uController1.6 (VBAT), uController1.95 (VDD33_USB), MR1.1, MnC11.2, MnC12.1, MnC13.1, MunC1.1, MunC2.1, SW1.1
- net at uController1.106 (VCAP): now also MbC4.1
- net BOOTSW: now reaches uController1.138 (BOOT0)
- net BOOTSW: now also SR1.2
- net RST_BTN: now reaches uController1.25 (NRST)
- net RST_BTN: now also B1.1, B1.2, BC1.1
- net at uController1.32 (VREF+): now also MR1.2, MbC2.1
- net at uController1.71 (VCAP): now also MbC3.1
- net at UR1.2: now also USB1.1
- new net: SR1.1, SW1.2
- no-connect marks 65 -> 69
