File: PCB_CAD/PCB_Order3/PCB_Order3.kicad_sch (KiCad schematic)
At the start: 93 parts, among them J1 Conn_01x03_Socket, SW1 SLW-883935-2A-D

Commit message: final schematic review minus debug ports (USB and SW)
Parts:
- Dac_DigitalSup_noise1, Dac_DigitalSup_noise2, DnC1, FnC1, FnC2, LLSIC1, LLSIC2, LnC1, RnC1, RnC2, RnC3, RnC4, RnC5, RnC6, RnC7: value 0.15u -> 0.1u
- DbC1: value 15u -> 10u
- J1: footprint Connector_PinSocket_2.54mm:PinSocket_1x03_P2.54mm_Vertical_SMD_Pin1Right -> Connector_PinSocket_2.54mm:PinSocket_1x03_P2.54mm_Vertical
- SPDIFR1, VDIVR1, VDIVR2: footprint Resistor_SMD:R_0603_1608Metric -> Resistor_SMD:R_0603_1608Metric_Pad0.98x0.95mm_HandSolder
- renumbered DCPEM to DCPEM1, LLSIN to LLSIN1, LLSOUT to LLSOUT1, RCAAin to RCAAin1, SPDIFTX to SPDIFTX1, TVS to TVS1
Connections:
- net GNDA: no longer uController1.31 (VSSA)
- net GNDD: now also uController1.31 (VSSA)
Changed lines of the file:
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@@
 			)
 		)
-		(property "Value" "0.15u"
+		(property "Value" "0.1u"
 			(at 510.794 290.83 90)
 			(effects
@@
 			)
 		)
-		(property "Value" "0.15u"
+		(property "Value" "0.1u"
 			(at 256.794 250.444 90)
 			(effects
@@
 			)
 		)
-		(property "Value" "0.15u"
+		(property "Value" "0.1u"
 			(at 597.916 334.264 0)
 			(effects
@@
 			)
 		)
-		(property "Value" "0.15u"
+		(property "Value" "0.1u"
 			(at 491.744 356.616 90)
 			(effects
@@
 			)
 		)
-		(property "Value" "0.15u"
+		(property "Value" "0.1u"
 			(at 305.054 250.698 90)
 			(effects
@@
 			)
 		)
-		(property "Footprint" "Connector_PinSocket_2.54mm:PinSocket_1x03_P2.54mm_Vertical_SMD_Pin1Right"
+		(property "Footprint" "Connector_PinSocket_2.54mm:PinSocket_1x03_P2.54mm_Vertical"
 			(at 237.49 304.8 0)
 			(effects
@@
 			)
 		)
-		(property "Value" "15u"
+		(property "Value" "10u"
 			(at 508 243.078 90)
 			(effects
@@
 			)
 		)
-		(property "Value" "0.15u"
+		(property "Value" "0.1u"
 			(at 670.814 328.422 90)
 			(effects
@@
 			)
 		)
-		(property "Value" "0.15u"
+		(property "Value" "0.1u"
 			(at 493.776 330.962 0)
 			(effects
@@
 		(on_board yes)
 		(dnp no)
-		(property "Reference" "LLSOUT"
+		(property "Reference" "LLSOUT1"
 			(at 687.578 197.612 0)
 			(effects
@@
 			(project ""
 				(path "/85a2a93a-53e0-46c8-b7f5-ee661b6f3053"
-					(reference "LLSOUT")
+					(reference "LLSOUT1")
 					(unit 1)
 				)
@@
 			)
 		)
-		(property "Value" "0.15u"
+		(property "Value" "0.1u"
 			(at 575.818 325.628 0)
 			(effects
@@
 			)
 		)
-		(property "Footprint" "Resistor_SMD:R_0603_1608Metric"
+		(property "Footprint" "Resistor_SMD:R_0603_1608Metric_Pad0.98x0.95mm_HandSolder"
 			(at 231.14 269.24 0)
 			(effects
@@
 			)
 		)
-		(property "Value" "0.15u"
+		(property "Value" "0.1u"
 			(at 496.57 318.262 0)
 			(effects
@@
 		(on_board yes)
 		(dnp no)
-		(property "Reference" "RCAAin"
+		(property "Reference" "RCAAin1"
 			(at 254.762 193.294 0)
 			(effects
@@
 			(project ""
 				(path "/85a2a93a-53e0-46c8-b7f5-ee661b6f3053"
-					(reference "RCAAin")
+					(reference "RCAAin1")
 					(unit 1)
 				)
@@
 			)
 		)
-		(property "Value" "0.15u"
+		(property "Value" "0.1u"
 			(at 591.566 274.574 0)
 			(effects
@@
 			)
 		)
-		(property "Footprint" "Resistor_SMD:R_0603_1608Metric"
+		(property "Footprint" "Resistor_SMD:R_0603_1608Metric_Pad0.98x0.95mm_HandSolder"
 			(at 237.49 323.85 0)
 			(effects
@@
 			)
 		)
-		(property "Value" "0.15u"
+		(property "Value" "0.1u"
 			(at 507.746 252.222 90)
 			(effects
@@
 			)
 		)
-		(property "Value" "0.15u"
+		(property "Value" "0.1u"
 			(at 575.564 310.134 0)
 			(effects
@@
 		(on_board yes)
 		(dnp no)
-		(property "Reference" "DCPEM"
+		(property "Reference" "DCPEM1"
 			(at 218.44 119.888 0)
 			(effects
@@
 			(project ""
 				(path "/85a2a93a-53e0-46c8-b7f5-ee661b6f3053"
-					(reference "DCPEM")
+					(reference "DCPEM1")
 					(unit 1)
 				)
@@
 	)
 	(symbol
-		(lib_id "power:GNDA")
+		(lib_id "power:GNDD")
 		(at 440.69 355.6 0)
 		(unit 1)
@@
 			)
 		)
-		(property "Value" "GNDA"
+		(property "Value" "GNDD"
 			(at 446.532 356.362 0)
 			(effects
@@
 			)
 		)
-		(property "Description" "Power symbol creates a global label with name \"GNDA\" , analog ground"
+		(property "Description" "Power symbol creates a global label with name \"GNDD\" , digital ground"
 			(at 440.69 355.6 0)
 			(effects
@@
 		(on_board yes)
 		(dnp no)
-		(property "Reference" "TVS"
+		(property "Reference" "TVS1"
 			(at 234.188 142.494 90)
 			(effects
@@
 			(project ""
 				(path "/85a2a93a-53e0-46c8-b7f5-ee661b6f3053"
-					(reference "TVS")
+					(reference "TVS1")
 					(unit 1)
 				)
@@
 			)
 		)
-		(property "Footprint" "Resistor_SMD:R_0603_1608Metric"
+		(property "Footprint" "Resistor_SMD:R_0603_1608Metric_Pad0.98x0.95mm_HandSolder"
 			(at 222.25 323.85 0)
 			(effects
@@
 			)
 		)
-		(property "Value" "0.15u"
+		(property "Value" "0.1u"
 			(at 338.074 297.434 90)
 			(effects
@@
 			)
 		)
-		(property "Value" "0.15u"
+		(property "Value" "0.1u"
 			(at 612.902 273.05 0)
 			(effects
@@
 		(on_board yes)
 		(dnp no)
-		(property "Reference" "LLSIN"
+		(property "Reference" "LLSIN1"
 			(at 279.908 262.89 0)
 			(effects
@@
 			(project ""
 				(path "/85a2a93a-53e0-46c8-b7f5-ee661b6f3053"
-					(reference "LLSIN")
+					(reference "LLSIN1")
 					(unit 1)
 				)
@@
 			)
 		)
-		(property "Value" "0.15u"
+		(property "Value" "0.1u"
 			(at 493.268 302.768 0)
 			(effects
@@
 		(on_board yes)
 		(dnp no)
-		(property "Reference" "SPDIFTX"
+		(property "Reference" "SPDIFTX1"
 			(at 582.676 198.882 0)
 			(effects
@@
 			(project ""
 				(path "/85a2a93a-53e0-46c8-b7f5-ee661b6f3053"
-					(reference "SPDIFTX")
+					(reference "SPDIFTX1")
 					(unit 1)
 				)

Commit message: change digital out blocks to use toslink
Parts:
- removed LLSIC1, LLSIC2, LLSOC1, LLSOC2, SPDIFC1, SPDIFC2: 0.1u, Capacitor_SMD:C_0805_2012Metric_Pad1.18x1.45mm_HandSolder, symbol Device:C_Small
- removed LLSIN1, LLSOUT1: SN74AXCH1T45DCKR, CustomModels:DCK6_TEX, symbol 2024-10-27_00-26-18:SN74AXCH1T45DCKR
- removed RCADin1, RCADout1: RCJ-027, CustomModels:CUI_RCJ-027, symbol RCJ-027:RCJ-027
- removed SPDIFR1, SPDIFR2: 75, Resistor_SMD:R_0603_1608Metric_Pad0.98x0.95mm_HandSolder, symbol Device:R_Small_US
- removed VDIVR1: 8.87k, Resistor_SMD:R_0603_1608Metric_Pad0.98x0.95mm_HandSolder, symbol Device:R_Small_US
- removed VDIVR2: 2.21k, Resistor_SMD:R_0603_1608Metric_Pad0.98x0.95mm_HandSolder, symbol Device:R_Small_US
- added LLSC1, LLSC2, LLSC3, LLSC4, TOSLINKC1, TOSLINKC2, USBC1: 0.1u, Capacitor_SMD:C_0805_2012Metric_Pad1.18x1.45mm_HandSolder, symbol Device:C_Small
- added LLSIN, LLSOUT: SN74LVC1T45DBVR, DBV0006A_N, symbol TI_LLS_50:SN74LVC1T45DBVR
- added TOSLINKIN: TORX1950A_F_, TORX1950AF, symbol TORX1950A_F_:TORX1950A_F_
- added TOSLINKL1: 47u, Inductor_SMD:L_10.4x10.4_H4.8, symbol Device:L_Small
- added TOSLINKOUT: TOTX1950A_F_, TOTX1950AF, symbol TOTX1950A_F_:TOTX1950A_F_
- added TOSLINKR1: 5.6k, Capacitor_SMD:C_0603_1608Metric_Pad1.08x0.95mm_HandSolder, symbol Device:R_Small_US
- added USBC2: 4.7u, Capacitor_THT:CP_Radial_D5.0mm_P2.00mm, symbol Device:C_Polarized_Small_US
Connections:
- net GNDA is gone; now on net GNDD: ADC1.4 (VSS), DAC1.1 (VSSA), DAC1.12 (LINEGND), RCAAin1.1, RCAAout1.1
- net GNDD: now also USB1.5, USB1.6 (MP1), USB1.7 (MP2), USB1.8 (MP3), USB1.9 (MP4), LLSC1.2, LLSC2.1, LLSC3.1, LLSC4.2, LLSIN.2 (GND), LLSIN.5 (DIR), LLSOUT.2 (GND), TOSLINKC1.2, TOSLINKC2.2, TOSLINKIN.2 (GND1), TOSLINKIN.4 (GND2), TOSLINKIN.MH1 (CASE_1), TOSLINKIN.MH2 (CASE_2), TOSLINKOUT.1 (GND), USBC1.2, USBC2.2
- net SPDIFRX_IN0: now also LLSIN.3 (A)
- net SPDIFTX_OUT: now also LLSOUT.3 (A)
- net VDD: now also LLSC1.1, LLSC3.2, LLSIN.1 (VCCA), LLSOUT.1 (VCCA), LLSOUT.5 (DIR)
- net VUSB: now reaches UR1.2, USB1.1
- net VUSB: now also LLSC2.2, LLSC4.1, LLSIN.6 (VCCB), LLSOUT.6 (VCCB), TOSLINKC2.1, TOSLINKL1.1, TOSLINKOUT.3 (VCC), TOSLINKR1.1, USBC1.1, USBC2.1
- new net: TOSLINKC1.1, TOSLINKIN.3 (VCC), TOSLINKL1.2
- new net: TOSLINKOUT.2 (_CURRENT_LIMITING_RESISTOR_OF_LED), TOSLINKR1.2
- new net SPDIF_RXOUT: LLSIN.4 (B), TOSLINKIN.1 (OUTPUT)
- new net TOSLINKTXIN: LLSOUT.4 (B), TOSLINKOUT.4 (INPUT)
- no-connect marks 104 -> 106
Other:
- note added: ":("
- note added: "Emergency Toslink"

Commit message: pcb emergency tosling complete. working on power
Parts:
- LLSIN1: renamed from LLSIN; footprint DBV0006A_N -> CustomModels:TI_LLS_50
- LLSOUT1: renamed from LLSOUT; footprint DBV0006A_N -> CustomModels:TI_LLS_50
- TOSLINKIN1: renamed from TOSLINKIN; footprint TORX1950AF -> CustomModels:TORX1950AF
- TOSLINKOUT1: renamed from TOSLINKOUT; footprint TOTX1950AF -> CustomModels:TOTX1950AF
Changed lines of the file:
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@@
 		(on_board yes)
 		(dnp no)
-		(property "Reference" "LLSIN"
+		(property "Reference" "LLSIN1"
 			(at 520.7 118.364 0)
 			(effects
@@
 			)
 		)
-		(property "Footprint" "DBV0006A_N"
+		(property "Footprint" "CustomModels:TI_LLS_50"
 			(at 521.97 119.38 0)
 			(effects
@@
 			(project ""
 				(path "/85a2a93a-53e0-46c8-b7f5-ee661b6f3053"
-					(reference "LLSIN")
+					(reference "LLSIN1")
 					(unit 1)
 				)
@@
 		(on_board yes)
 		(dnp no)
-		(property "Reference" "TOSLINKOUT"
+		(property "Reference" "TOSLINKOUT1"
 			(at 584.454 133.096 0)
 			(effects
@@
 			)
 		)
-		(property "Footprint" "TOTX1950AF"
+		(property "Footprint" "CustomModels:TOTX1950AF"
 			(at 613.41 232.08 0)
 			(effects
@@
 			(project ""
 				(path "/85a2a93a-53e0-46c8-b7f5-ee661b6f3053"
-					(reference "TOSLINKOUT")
+					(reference "TOSLINKOUT1")
 					(unit 1)
 				)
@@
 		(on_board yes)
 		(dnp no)
-		(property "Reference" "TOSLINKIN"
+		(property "Reference" "TOSLINKIN1"
 			(at 585.216 92.202 0)
 			(effects
@@
 			)
 		)
-		(property "Footprint" "TORX1950AF"
+		(property "Footprint" "CustomModels:TORX1950AF"
 			(at 598.17 191.44 0)
 			(effects
@@
 			(project ""
 				(path "/85a2a93a-53e0-46c8-b7f5-ee661b6f3053"
-					(reference "TOSLINKIN")
+					(reference "TOSLINKIN1")
 					(unit 1)
 				)
@@
 		(on_board yes)
 		(dnp no)
-		(property "Reference" "LLSOUT"
+		(property "Reference" "LLSOUT1"
 			(at 662.432 136.652 0)
 			(effects
@@
 			)
 		)
-		(property "Footprint" "DBV0006A_N"
+		(property "Footprint" "CustomModels:TI_LLS_50"
 			(at 662.94 137.16 0)
 			(effects
@@
 			(project ""
 				(path "/85a2a93a-53e0-46c8-b7f5-ee661b6f3053"
-					(reference "LLSOUT")
+					(reference "LLSOUT1")
 					(unit 1)
 				)
